Commit message: Update basic_amr1.urdf

File: urdf/basic_amr1.urdf (robot description, URDF)
Before this commit: robot basic_amr, 2 links, 1 joints
Links:
- removed link base
- added link base_footprint
- link base_link: geometry visual box size=0.08 0.05 0.002
Joints:
- removed joint base__base_link
- added joint base_link__base_footprint: type fixed, parent base_footprint, child base_link
