Commit message: Update basic_amr_gazebo.urdf

File: urdf/basic_amr_gazebo.urdf (robot description, URDF)
Before this commit: robot basic_amr, 6 links, 5 joints
Links:
- removed link base
- added link base_footprint
- link base_link: mass None -> 0.5; geometry collision box size=0.08 0.05 0.002; visual box size=0.08 0.05 0.002
Joints:
- removed joint base__base_link
- removed joint base__bcastor_wheel
- removed joint base__fcastor_wheel
- added joint base_footprint__base_link: type fixed, parent base_footprint, child base_link
- added joint base_link__bcastor_wheel: type continuous, parent base_link, child bcastor_wheel, origin xyz=-0.028 0 -0.005 rpy=1.5708 0 0, axis 0 0 1
- added joint base_link__fcastor_wheel: type continuous, parent base_link, child fcastor_wheel, origin xyz=0.028 0 -0.005 rpy=1.5708 0 0, axis 0 0 1
- joint wheel_left_joint: parent base -> base_link
- joint wheel_right_joint: parent base -> base_link
